File: examples/emc-flyback-demo/design/emc_flyback.kicad_sch (KiCad schematic)
At the start: 88 parts, among them J1 VIN+ 24V, J2 VIN- 0V, J3 VOUT +12V, J4 VOUT 0V, J5 CHASSIS, Q1 IRF520NPBF, T1 750311591, U1 UC3845B, U2 L78L12ACUTR, U3 TL431AIDBZR, U4 LTV-817S

Commit message: Remove course code from text files and note the board was designed with Claude
Co-authored-by: Cursor <cursoragent@cursor.com>
Other:
- company: TU/e EPE - 5SWB0 Advanced Power Electronics -> TU/e EPE
Changed lines of the file:
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@@
 (kicad_sch (version 20230121) (generator eeschema)
   (paper "A3")
-  (title_block (title "EMC teaching demo - 24V/12V flyback with EMC knobs") (date "2026-10-03") (rev "D") (company "TU/e EPE - 5SWB0 Advanced Power Electronics") (comment 1 "Generated with Claude; verify before ordering"))
+  (title_block (title "EMC teaching demo - 24V/12V flyback with EMC knobs") (date "2026-10-03") (rev "D") (company "TU/e EPE") (comment 1 "Generated with Claude; verify before ordering"))
   (symbol (lib_id "Connector_Generic:Conn_01x01") (at 22.86 50.8 180) (unit 1) (in_bom yes) (on_board yes) (dnp no)
     (property "Reference" "J1" (at 22.86 53.34 0) (effects (font (size 1.27 1.27))))
